Commit message: feat: Update controllers to use velocity control and enhance steering dynamics
Co-authored-by: Copilot <copilot@github.com>

File: boa_new_urdf_description/urdf/boa_new_urdf.xacro (robot description, xacro)
@@ -249,6 +249,6 @@
   <child link="direction_motor_1"/>
   <axis xyz="0.0 0.0 1.0"/>
-  <limit lower="-1.5707" upper="1.5707" effort="100.0" velocity="1.0"/>
-  <dynamics damping="10.0" friction="1.0"/>
+  <limit lower="-1.5707" upper="1.5707" effort="500.0" velocity="5.0"/>
+  <dynamics damping="0.5" friction="0.0"/>
 </joint>
 <joint name="lift_joint" type="prismatic">
@@ -303,7 +303,7 @@
   </hardware>
   <joint name="direction_motor_joint">
-    <command_interface name="position">
-      <param name="min">-1.5707</param>
-      <param name="max">1.5707</param>
+    <command_interface name="velocity">
+      <param name="min">-5.0</param>
+      <param name="max">5.0</param>
     </command_interface>
     <state_interface name="position">

Commit message: fix: Adjust joint limits in URDF and enhance Kinco drive node logging
Co-authored-by: Copilot <copilot@github.com>

File: boa_new_urdf_description/urdf/boa_new_urdf.xacro (robot description, xacro)
@@ -249,5 +249,5 @@
   <child link="direction_motor_1"/>
   <axis xyz="0.0 0.0 1.0"/>
-  <limit lower="-1.5707" upper="1.5707" effort="500.0" velocity="5.0"/>
+  <limit lower="-1.5708" upper="1.5708" effort="500.0" velocity="5.0"/>
   <dynamics damping="0.5" friction="0.0"/>
 </joint>

Commit message: feat: Add traction slew rate control and update traction command logic in Kinco drive node
Co-authored-by: Copilot <copilot@github.com>

File: boa_new_urdf_description/urdf/boa_new_urdf.xacro (robot description, xacro)
@@ -243,4 +243,5 @@
   <child link="drive_motor_1"/>
   <axis xyz="0.0 1.0 0.0"/>
+  <dynamics damping="0.3" friction="0.0"/>
 </joint>
 <joint name="direction_motor_joint" type="revolute">

Commit message: feat: Update URDF and launch files for improved localization and mapping configuration
Co-authored-by: Copilot <copilot@github.com>

File: boa_new_urdf_description/urdf/boa_new_urdf.xacro (robot description, xacro)
@@ -4,4 +4,10 @@
 <xacro:include filename="$(find boa_new_urdf_description)/urdf/boa_new_urdf.trans" />
 <xacro:include filename="$(find boa_new_urdf_description)/urdf/boa_new_urdf.gazebo" />
+<link name="base_footprint"/>
+<joint name="base_footprint_joint" type="fixed">
+  <origin xyz="0 0 0" rpy="0 0 0"/>
+  <parent link="base_footprint"/>
+  <child link="base_link"/>
+</joint>
 <link name="base_link">
   <inertial>

Commit message: feat: Enhance dynamics properties for caster and drive motor joints in URDF
Co-authored-by: Copilot <copilot@github.com>

File: boa_new_urdf_description/urdf/boa_new_urdf.xacro (robot description, xacro)
@@ -237,4 +237,5 @@
   <child link="right_caster_1"/>
   <axis xyz="0.0 1.0 0.0"/>
+  <dynamics damping="1.5" friction="0.5"/>
 </joint>
 <joint name="left_caster_joint" type="continuous">
@@ -243,4 +244,5 @@
   <child link="left_caster_1"/>
   <axis xyz="-0.0 -1.0 0.0"/>
+  <dynamics damping="1.5" friction="0.5"/>
 </joint>
 <joint name="drive_motor_joint" type="continuous">
@@ -257,5 +259,5 @@
   <axis xyz="0.0 0.0 1.0"/>
   <limit lower="-1.5708" upper="1.5708" effort="500.0" velocity="5.0"/>
-  <dynamics damping="0.5" friction="0.0"/>
+  <dynamics damping="5.0" friction="0.5"/>
 </joint>
 <joint name="lift_joint" type="prismatic">

Commit message: refactor: Update inertial properties and friction parameters for drive and direction motors
Co-authored-by: Copilot <copilot@github.com>

File: boa_new_urdf_description/urdf/boa_new_urdf.xacro (robot description, xacro)
@@ -12,7 +12,7 @@
 <link name="base_link">
   <inertial>
-    <origin xyz="0.945398072688781 -0.001011453583043792 1.1145363303175833" rpy="0 0 0"/>
-    <mass value="781.2318135532329"/>
-    <inertia ixx="196.374943" iyy="188.293374" izz="40.387878" ixy="0.085427" iyz="-0.535549" ixz="-13.126993"/>
+    <origin xyz="0.945398072688781 -0.001011453583043792 0.1" rpy="0 0 0"/>
+    <mass value="60.0"/>
+    <inertia ixx="15.121" iyy="14.499" izz="3.110" ixy="0.007" iyz="-0.041" ixz="-1.011"/>
   </inertial>
   <visual>
@@ -258,5 +258,5 @@
   <child link="direction_motor_1"/>
   <axis xyz="0.0 0.0 1.0"/>
-  <limit lower="-1.5708" upper="1.5708" effort="500.0" velocity="5.0"/>
+  <limit lower="-1.5708" upper="1.5708" effort="300.0" velocity="0.8"/>
   <dynamics damping="5.0" friction="0.5"/>
 </joint>

Commit message: refactor: Update collision geometry for caster links and adjust self-collision settings
Co-authored-by: Copilot <copilot@github.com>

File: boa_new_urdf_description/urdf/boa_new_urdf.xacro (robot description, xacro)
@@ -44,7 +44,7 @@
   </visual>
   <collision>
-    <origin xyz="-0.0 0.275 -0.04" rpy="0 0 0"/>
-    <geometry>
-      <mesh filename="file://$(find boa_new_urdf_description)/meshes/right_caster_1.stl" scale="0.001 0.001 0.001"/>
+    <origin xyz="0.0 0.275 -0.04" rpy="0 0 0"/>
+    <geometry>
+      <sphere radius="0.04"/>
     </geometry>
   </collision>
@@ -64,7 +64,7 @@
   </visual>
   <collision>
-    <origin xyz="-0.0 -0.275 -0.04" rpy="0 0 0"/>
-    <geometry>
-      <mesh filename="file://$(find boa_new_urdf_description)/meshes/left_caster_1.stl" scale="0.001 0.001 0.001"/>
+    <origin xyz="0.0 -0.275 -0.04" rpy="0 0 0"/>
+    <geometry>
+      <sphere radius="0.04"/>
     </geometry>
   </collision>

Commit message: refactor: Update dynamics parameters for direction motor joint to improve performance
Co-authored-by: Copilot <copilot@github.com>

File: boa_new_urdf_description/urdf/boa_new_urdf.xacro (robot description, xacro)
@@ -258,6 +258,6 @@
   <child link="direction_motor_1"/>
   <axis xyz="0.0 0.0 1.0"/>
-  <limit lower="-1.5708" upper="1.5708" effort="300.0" velocity="0.8"/>
-  <dynamics damping="5.0" friction="0.5"/>
+  <limit lower="-1.5708" upper="1.5708" effort="300.0" velocity="1.2"/>
+  <dynamics damping="3.0" friction="0.5"/>
 </joint>
 <joint name="lift_joint" type="prismatic">

Commit message: refactor: Update URDF and launch files for improved localization and steering control
Co-authored-by: Copilot <copilot@github.com>

File: boa_new_urdf_description/urdf/boa_new_urdf.xacro (robot description, xacro)
@@ -12,7 +12,7 @@
 <link name="base_link">
   <inertial>
-    <origin xyz="0.945398072688781 -0.001011453583043792 0.1" rpy="0 0 0"/>
-    <mass value="60.0"/>
-    <inertia ixx="15.121" iyy="14.499" izz="3.110" ixy="0.007" iyz="-0.041" ixz="-1.011"/>
+    <origin xyz="0.945398072688781 -0.001011453583043792 1.1145363303175833" rpy="0 0 0"/>
+    <mass value="781.2318135532329"/>
+    <inertia ixx="196.374943" iyy="188.293374" izz="40.387878" ixy="0.085427" iyz="-0.535549" ixz="-13.126993"/>
   </inertial>
   <visual>
@@ -44,7 +44,7 @@
   </visual>
   <collision>
-    <origin xyz="0.0 0.275 -0.04" rpy="0 0 0"/>
-    <geometry>
-      <sphere radius="0.04"/>
+    <origin xyz="-0.0 0.275 -0.04" rpy="0 0 0"/>
+    <geometry>
+      <mesh filename="file://$(find boa_new_urdf_description)/meshes/right_caster_1.stl" scale="0.001 0.001 0.001"/>
     </geometry>
   </collision>
@@ -64,7 +64,7 @@
   </visual>
   <collision>
-    <origin xyz="0.0 -0.275 -0.04" rpy="0 0 0"/>
-    <geometry>
-      <sphere radius="0.04"/>
+    <origin xyz="-0.0 -0.275 -0.04" rpy="0 0 0"/>
+    <geometry>
+      <mesh filename="file://$(find boa_new_urdf_description)/meshes/left_caster_1.stl" scale="0.001 0.001 0.001"/>
     </geometry>
   </collision>
@@ -258,6 +258,6 @@
   <child link="direction_motor_1"/>
   <axis xyz="0.0 0.0 1.0"/>
-  <limit lower="-1.5708" upper="1.5708" effort="300.0" velocity="1.2"/>
-  <dynamics damping="3.0" friction="0.5"/>
+  <limit lower="-1.5708" upper="1.5708" effort="500.0" velocity="5.0"/>
+  <dynamics damping="5.0" friction="0.5"/>
 </joint>
 <joint name="lift_joint" type="prismatic">

Commit message: fix: Adjust LIDAR scan parameters and update lidar_fork_joint origin for improved accuracy
Co-authored-by: Copilot <copilot@github.com>

File: boa_new_urdf_description/urdf/boa_new_urdf.xacro (robot description, xacro)
@@ -270,5 +270,5 @@
 </joint>
 <joint name="lidar_fork_joint" type="fixed">
-  <origin xyz="-0.45 -0.235 0.0685" rpy="0 0 0"/>
+  <origin xyz="-0.45 -0.235 0.06" rpy="0 0 3.14159265"/>
   <parent link="base_link"/>
   <child link="lidar_fork_1"/>

Commit message: fix: Update lidar_fork_joint origin and adjust pallet detection parameters for improved accuracy
Co-authored-by: Copilot <copilot@github.com>

File: boa_new_urdf_description/urdf/boa_new_urdf.xacro (robot description, xacro)
@@ -270,5 +270,5 @@
 </joint>
 <joint name="lidar_fork_joint" type="fixed">
-  <origin xyz="-0.45 -0.235 0.06" rpy="0 0 3.14159265"/>
+  <origin xyz="-0.45 -0.235 0.05" rpy="0 0 3.14159265"/>
   <parent link="base_link"/>
   <child link="lidar_fork_1"/>

Commit message: fix: Correct drive motor joint origin position and update comments for clarity
Co-authored-by: Copilot <copilot@github.com>

File: boa_new_urdf_description/urdf/boa_new_urdf.xacro (robot description, xacro)
@@ -247,5 +247,5 @@
 </joint>
 <joint name="drive_motor_joint" type="continuous">
-  <origin xyz="0.0057 0.0 -0.2255" rpy="0 0 -1.5707963"/>
+  <origin xyz="0.0 0.0 -0.2255" rpy="0 0 -1.5707963"/>
   <parent link="direction_motor_1"/>
   <child link="drive_motor_1"/>
