Commit message: feat: Update URDF and launch files for improved robot model configuration

File: boa_new_urdf_description/urdf/boa_new_urdf.xacro (robot description, xacro)
@@ -66,10 +66,10 @@
 <link name="drive_motor_1">
   <inertial>
-    <origin xyz="1.919312224924131 1.629849831257866e-08 -4.287126238095018e-06" rpy="0 0 0"/>
+    <origin xyz="-0.012752 0.0 0.000696" rpy="0 0 0"/>
     <mass value="17.21864059844125"/>
     <inertia ixx="0.124174" iyy="0.072747" izz="0.072745" ixy="-0.0" iyz="-0.0" ixz="-3e-06"/>
   </inertial>
   <visual>
-    <origin xyz="0.830664 0.0 -0.109" rpy="0 0 0"/>
+    <origin xyz="-1.1014 0.0 -0.1083" rpy="0 0 0"/>
     <geometry>
       <mesh filename="file://$(find boa_new_urdf_description)/meshes/drive_motor_1.stl" scale="0.001 0.001 0.001"/>
@@ -78,5 +78,5 @@
   </visual>
   <collision>
-    <origin xyz="0.830664 0.0 -0.109" rpy="0 0 0"/>
+    <origin xyz="-1.1014 0.0 -0.1083" rpy="0 0 0"/>
     <geometry>
       <mesh filename="file://$(find boa_new_urdf_description)/meshes/drive_motor_1.stl" scale="0.001 0.001 0.001"/>
@@ -86,10 +86,10 @@
 <link name="direction_motor_1">
   <inertial>
-    <origin xyz="1.1675247319514686 -0.0002473749983548974 -0.065560452505046" rpy="0 0 0"/>
+    <origin xyz="0.054600 -0.000200 -0.092060" rpy="0 0 0"/>
     <mass value="20.417319679069678"/>
     <inertia ixx="0.182357" iyy="0.193956" izz="0.141973" ixy="-0.000532" iyz="0.001583" ixz="0.045478"/>
   </inertial>
   <visual>
-    <origin xyz="0.045716 0.0 -0.308" rpy="0 0 0"/>
+    <origin xyz="-1.1129 0.0 -0.3345" rpy="0 0 0"/>
     <geometry>
       <mesh filename="file://$(find boa_new_urdf_description)/meshes/direction_motor_1.stl" scale="0.001 0.001 0.001"/>
@@ -98,5 +98,5 @@
   </visual>
   <collision>
-    <origin xyz="0.045716 0.0 -0.308" rpy="0 0 0"/>
+    <origin xyz="-1.1129 0.0 -0.3345" rpy="0 0 0"/>
     <geometry>
       <mesh filename="file://$(find boa_new_urdf_description)/meshes/direction_motor_1.stl" scale="0.001 0.001 0.001"/>
@@ -237,5 +237,5 @@
 </joint>
 <joint name="drive_motor_joint" type="continuous">
-  <origin xyz="-0.784948 0.0 -0.199" rpy="0 0 0"/>
+  <origin xyz="-0.0115 0.0 -0.2262" rpy="0 0 0"/>
   <parent link="direction_motor_1"/>
   <child link="drive_motor_1"/>
@@ -243,8 +243,8 @@
 </joint>
 <joint name="direction_motor_joint" type="continuous">
-  <origin xyz="-0.045716 0.0 0.308" rpy="0 0 0"/>
+  <origin xyz="1.1129 0.0 0.3345" rpy="0 0 0"/>
   <parent link="base_link"/>
   <child link="direction_motor_1"/>
-  <axis xyz="-0.0 0.0 -1.0"/>
+  <axis xyz="0.0 0.0 1.0"/>
 </joint>
 <joint name="lift_joint" type="fixed">

Commit message: fix: Adjust inertial and joint origin parameters for drive and direction motors

File: boa_new_urdf_description/urdf/boa_new_urdf.xacro (robot description, xacro)
@@ -66,5 +66,5 @@
 <link name="drive_motor_1">
   <inertial>
-    <origin xyz="-0.012752 0.0 0.000696" rpy="0 0 0"/>
+    <origin xyz="-0.012700 0.0 0.000700" rpy="0 0 0"/>
     <mass value="17.21864059844125"/>
     <inertia ixx="0.124174" iyy="0.072747" izz="0.072745" ixy="-0.0" iyz="-0.0" ixz="-3e-06"/>
@@ -86,10 +86,10 @@
 <link name="direction_motor_1">
   <inertial>
-    <origin xyz="0.054600 -0.000200 -0.092060" rpy="0 0 0"/>
+    <origin xyz="0.066100 -0.000200 -0.092060" rpy="0 0 0"/>
     <mass value="20.417319679069678"/>
     <inertia ixx="0.182357" iyy="0.193956" izz="0.141973" ixy="-0.000532" iyz="0.001583" ixz="0.045478"/>
   </inertial>
   <visual>
-    <origin xyz="-1.1129 0.0 -0.3345" rpy="0 0 0"/>
+    <origin xyz="-1.1014 0.0 -0.3345" rpy="0 0 0"/>
     <geometry>
       <mesh filename="file://$(find boa_new_urdf_description)/meshes/direction_motor_1.stl" scale="0.001 0.001 0.001"/>
@@ -98,5 +98,5 @@
   </visual>
   <collision>
-    <origin xyz="-1.1129 0.0 -0.3345" rpy="0 0 0"/>
+    <origin xyz="-1.1014 0.0 -0.3345" rpy="0 0 0"/>
     <geometry>
       <mesh filename="file://$(find boa_new_urdf_description)/meshes/direction_motor_1.stl" scale="0.001 0.001 0.001"/>
@@ -237,5 +237,5 @@
 </joint>
 <joint name="drive_motor_joint" type="continuous">
-  <origin xyz="-0.0115 0.0 -0.2262" rpy="0 0 0"/>
+  <origin xyz="0.0 0.0 -0.2262" rpy="0 0 0"/>
   <parent link="direction_motor_1"/>
   <child link="drive_motor_1"/>
@@ -243,5 +243,5 @@
 </joint>
 <joint name="direction_motor_joint" type="continuous">
-  <origin xyz="1.1129 0.0 0.3345" rpy="0 0 0"/>
+  <origin xyz="1.1014 0.0 0.3345" rpy="0 0 0"/>
   <parent link="base_link"/>
   <child link="direction_motor_1"/>

Commit message: fix: Update inertial and joint origin parameters for direction motor and drive motor

File: boa_new_urdf_description/urdf/boa_new_urdf.xacro (robot description, xacro)
@@ -86,10 +86,10 @@
 <link name="direction_motor_1">
   <inertial>
-    <origin xyz="0.066100 -0.000200 -0.092060" rpy="0 0 0"/>
+    <origin xyz="0.071800 -0.000200 -0.092100" rpy="0 0 0"/>
     <mass value="20.417319679069678"/>
     <inertia ixx="0.182357" iyy="0.193956" izz="0.141973" ixy="-0.000532" iyz="0.001583" ixz="0.045478"/>
   </inertial>
   <visual>
-    <origin xyz="-1.1014 0.0 -0.3345" rpy="0 0 0"/>
+    <origin xyz="-1.0957 0.0 -0.3345" rpy="0 0 0"/>
     <geometry>
       <mesh filename="file://$(find boa_new_urdf_description)/meshes/direction_motor_1.stl" scale="0.001 0.001 0.001"/>
@@ -98,5 +98,5 @@
   </visual>
   <collision>
-    <origin xyz="-1.1014 0.0 -0.3345" rpy="0 0 0"/>
+    <origin xyz="-1.0957 0.0 -0.3345" rpy="0 0 0"/>
     <geometry>
       <mesh filename="file://$(find boa_new_urdf_description)/meshes/direction_motor_1.stl" scale="0.001 0.001 0.001"/>
@@ -237,5 +237,5 @@
 </joint>
 <joint name="drive_motor_joint" type="continuous">
-  <origin xyz="0.0 0.0 -0.2262" rpy="0 0 0"/>
+  <origin xyz="0.0057 0.0 -0.2262" rpy="0 0 0"/>
   <parent link="direction_motor_1"/>
   <child link="drive_motor_1"/>
@@ -243,5 +243,5 @@
 </joint>
 <joint name="direction_motor_joint" type="continuous">
-  <origin xyz="1.1014 0.0 0.3345" rpy="0 0 0"/>
+  <origin xyz="1.0957 0.0 0.3345" rpy="0 0 0"/>
   <parent link="base_link"/>
   <child link="direction_motor_1"/>

Commit message: fix: Adjust origin parameters for drive motor and drive motor joint

File: boa_new_urdf_description/urdf/boa_new_urdf.xacro (robot description, xacro)
@@ -66,10 +66,10 @@
 <link name="drive_motor_1">
   <inertial>
-    <origin xyz="-0.012700 0.0 0.000700" rpy="0 0 0"/>
+    <origin xyz="-0.012700 0.0 0.000004" rpy="0 0 0"/>
     <mass value="17.21864059844125"/>
     <inertia ixx="0.124174" iyy="0.072747" izz="0.072745" ixy="-0.0" iyz="-0.0" ixz="-3e-06"/>
   </inertial>
   <visual>
-    <origin xyz="-1.1014 0.0 -0.1083" rpy="0 0 0"/>
+    <origin xyz="-1.1014 0.0 -0.10899" rpy="0 0 0"/>
     <geometry>
       <mesh filename="file://$(find boa_new_urdf_description)/meshes/drive_motor_1.stl" scale="0.001 0.001 0.001"/>
@@ -78,5 +78,5 @@
   </visual>
   <collision>
-    <origin xyz="-1.1014 0.0 -0.1083" rpy="0 0 0"/>
+    <origin xyz="-1.1014 0.0 -0.10899" rpy="0 0 0"/>
     <geometry>
       <mesh filename="file://$(find boa_new_urdf_description)/meshes/drive_motor_1.stl" scale="0.001 0.001 0.001"/>
@@ -237,5 +237,5 @@
 </joint>
 <joint name="drive_motor_joint" type="continuous">
-  <origin xyz="0.0057 0.0 -0.2262" rpy="0 0 0"/>
+  <origin xyz="0.0057 0.0 -0.2255" rpy="0 0 0"/>
   <parent link="direction_motor_1"/>
   <child link="drive_motor_1"/>

Commit message: feat: Add cmd_vel relay node and update launch/config files for tricycle controller

File: boa_new_urdf_description/urdf/boa_new_urdf.xacro (robot description, xacro)
@@ -278,3 +278,24 @@
   <child link="case_1"/>
 </joint>
+<ros2_control name="boa_hardware" type="system">
+  <hardware>
+    <plugin>gz_ros2_control/GazeboSimSystem</plugin>
+  </hardware>
+  <joint name="direction_motor_joint">
+    <command_interface name="position">
+      <param name="min">-1.5707</param>
+      <param name="max">1.5707</param>
+    </command_interface>
+    <state_interface name="position"/>
+    <state_interface name="velocity"/>
+  </joint>
+  <joint name="drive_motor_joint">
+    <command_interface name="velocity">
+      <param name="min">-5.0</param>
+      <param name="max">5.0</param>
+    </command_interface>
+    <state_interface name="position"/>
+    <state_interface name="velocity"/>
+  </joint>
+</ros2_control>
 </robot>

Commit message: fix: Update friction parameters and joint types for improved robot dynamics

File: boa_new_urdf_description/urdf/boa_new_urdf.xacro (robot description, xacro)
@@ -78,7 +78,9 @@
   </visual>
   <collision>
-    <origin xyz="-1.1014 0.0 -0.10899" rpy="0 0 0"/>
-    <geometry>
-      <mesh filename="file://$(find boa_new_urdf_description)/meshes/drive_motor_1.stl" scale="0.001 0.001 0.001"/>
+    <!-- Cylinder collision for proper rolling contact in Gazebo -->
+    <!-- Wheel axle is X axis in this frame; URDF cylinder default is Z, so rotate 90° around Y -->
+    <origin xyz="0 0 0" rpy="0 1.5707963 0"/>
+    <geometry>
+      <cylinder radius="0.109" length="0.145"/>
     </geometry>
   </collision>
@@ -242,9 +244,11 @@
   <axis xyz="1.0 0.0 -0.0"/>
 </joint>
-<joint name="direction_motor_joint" type="continuous">
+<joint name="direction_motor_joint" type="revolute">
   <origin xyz="1.0957 0.0 0.3345" rpy="0 0 0"/>
   <parent link="base_link"/>
   <child link="direction_motor_1"/>
   <axis xyz="0.0 0.0 1.0"/>
+  <limit lower="-1.5707" upper="1.5707" effort="100.0" velocity="1.0"/>
+  <dynamics damping="10.0" friction="1.0"/>
 </joint>
 <joint name="lift_joint" type="fixed">
@@ -287,5 +291,7 @@
       <param name="max">1.5707</param>
     </command_interface>
-    <state_interface name="position"/>
+    <state_interface name="position">
+      <param name="initial_value">0.0</param>
+    </state_interface>
     <state_interface name="velocity"/>
   </joint>

Commit message: fix: Correct collision cylinder orientation and joint axis for proper robot dynamics

File: boa_new_urdf_description/urdf/boa_new_urdf.xacro (robot description, xacro)
@@ -79,6 +79,6 @@
   <collision>
     <!-- Cylinder collision for proper rolling contact in Gazebo -->
-    <!-- Wheel axle is X axis in this frame; URDF cylinder default is Z, so rotate 90° around Y -->
-    <origin xyz="0 0 0" rpy="0 1.5707963 0"/>
+    <!-- Wheel rolls in X direction: cylinder axis = Y, rotate Z→Y (90° around X) -->
+    <origin xyz="0 0 0" rpy="1.5707963 0 0"/>
     <geometry>
       <cylinder radius="0.109" length="0.145"/>
@@ -242,5 +242,5 @@
   <parent link="direction_motor_1"/>
   <child link="drive_motor_1"/>
-  <axis xyz="1.0 0.0 -0.0"/>
+  <axis xyz="0.0 1.0 0.0"/>
 </joint>
 <joint name="direction_motor_joint" type="revolute">

Commit message: fix: Rename slamware references to lidar_top for consistency in URDF files

File: boa_new_urdf_description/urdf/boa_new_urdf.xacro (robot description, xacro)
@@ -186,5 +186,5 @@
   </collision>
 </link>
-<link name="slamware_1">
+<link name="lidar_top">
   <inertial>
     <origin xyz="-4.3560027251920985e-06 4.649845288881102e-06 0.03323324367886471" rpy="0 0 0"/>
@@ -275,5 +275,5 @@
   <origin xyz="0.84 -2.6e-05 2.051002" rpy="0 0 0"/>
   <parent link="base_link"/>
-  <child link="slamware_1"/>
+  <child link="lidar_top"/>
 </joint>
 <joint name="case_joint" type="fixed">

Commit message: feat: Add IMU sensor integration and update launch configuration for improved robot dynamics

File: boa_new_urdf_description/urdf/boa_new_urdf.xacro (robot description, xacro)
@@ -276,4 +276,17 @@
   <parent link="base_link"/>
   <child link="lidar_top"/>
+</joint>
+<link name="imu_link">
+  <inertial>
+    <origin xyz="0 0 0" rpy="0 0 0"/>
+    <mass value="0.001"/>
+    <inertia ixx="1e-06" iyy="1e-06" izz="1e-06" ixy="0" iyz="0" ixz="0"/>
+  </inertial>
+</link>
+<joint name="imu_joint" type="fixed">
+  <!-- Same position as lidar_top -->
+  <origin xyz="0.84 -2.6e-05 2.051002" rpy="0 0 0"/>
+  <parent link="base_link"/>
+  <child link="imu_link"/>
 </joint>
 <joint name="case_joint" type="fixed">

Commit message: feat: Add lift controller and update URDF for lift joint dynamics

File: boa_new_urdf_description/urdf/boa_new_urdf.xacro (robot description, xacro)
@@ -252,8 +252,11 @@
   <dynamics damping="10.0" friction="1.0"/>
 </joint>
-<joint name="lift_joint" type="fixed">
+<joint name="lift_joint" type="prismatic">
   <origin xyz="0.82 0.0 0.07" rpy="0 0 0"/>
   <parent link="base_link"/>
   <child link="lift_1"/>
+  <axis xyz="0.0 0.0 1.0"/>
+  <limit lower="0.0" upper="1.5" effort="5000.0" velocity="0.2"/>
+  <dynamics damping="500.0" friction="100.0"/>
 </joint>
 <joint name="lidar_fork_joint" type="fixed">
@@ -317,4 +320,14 @@
     <state_interface name="velocity"/>
   </joint>
+  <joint name="lift_joint">
+    <command_interface name="position">
+      <param name="min">0.0</param>
+      <param name="max">1.5</param>
+    </command_interface>
+    <state_interface name="position">
+      <param name="initial_value">0.0</param>
+    </state_interface>
+    <state_interface name="velocity"/>
+  </joint>
 </ros2_control>
 </robot>

Commit message: fix: Adjust visual and joint origins for drive motor alignment

File: boa_new_urdf_description/urdf/boa_new_urdf.xacro (robot description, xacro)
@@ -71,5 +71,5 @@
   </inertial>
   <visual>
-    <origin xyz="-1.1014 0.0 -0.10899" rpy="0 0 0"/>
+    <origin xyz="0.0 -1.1014 -0.10899" rpy="0 0 1.5707963"/>
     <geometry>
       <mesh filename="file://$(find boa_new_urdf_description)/meshes/drive_motor_1.stl" scale="0.001 0.001 0.001"/>
@@ -239,5 +239,5 @@
 </joint>
 <joint name="drive_motor_joint" type="continuous">
-  <origin xyz="0.0057 0.0 -0.2255" rpy="0 0 0"/>
+  <origin xyz="0.0057 0.0 -0.2255" rpy="0 0 -1.5707963"/>
   <parent link="direction_motor_1"/>
   <child link="drive_motor_1"/>

Commit message: fix: Update direction motor joint orientation for correct alignment

File: boa_new_urdf_description/urdf/boa_new_urdf.xacro (robot description, xacro)
@@ -245,5 +245,5 @@
 </joint>
 <joint name="direction_motor_joint" type="revolute">
-  <origin xyz="1.0957 0.0 0.3345" rpy="0 0 0"/>
+  <origin xyz="1.0957 0.0 0.3345" rpy="0 0 1.5707963"/>
   <parent link="base_link"/>
   <child link="direction_motor_1"/>

Commit message: big commit

File: boa_new_urdf_description/urdf/boa_new_urdf.xacro (robot description, xacro)
@@ -270,5 +270,5 @@
 </joint>
 <joint name="lidar_fork_joint" type="fixed">
-  <origin xyz="-0.45 -0.235 0.05" rpy="0 0 3.14159265"/>
+  <origin xyz="-0.45 -0.235 0.05" rpy="0 0 0"/>
   <parent link="base_link"/>
   <child link="lidar_fork_1"/>
