Commit message: Update lidar joint orientations for correct alignment

File: robot_description/boa_new_urdf_description/urdf/boa_new_urdf.xacro (robot description, xacro)
@@ -275,10 +275,10 @@
 </joint>
 <joint name="lidar_left_joint" type="fixed">
-  <origin xyz="1.29 0.313 0.086" rpy="0 0 0"/>
+  <origin xyz="1.29 0.313 0.086" rpy="0 0 1.5707963"/>
   <parent link="base_link"/>
   <child link="lidar_left_1"/>
 </joint>
 <joint name="lidar_right_joint" type="fixed">
-  <origin xyz="1.29 -0.313 0.086" rpy="0 0 0"/>
+  <origin xyz="1.29 -0.313 0.086" rpy="0 0 1.5707963"/>
   <parent link="base_link"/>
   <child link="lidar_right_1"/>

Commit message: Update Lidar configurations for improved accuracy and adjust scan angle filters

File: robot_description/boa_new_urdf_description/urdf/boa_new_urdf.xacro (robot description, xacro)
@@ -275,5 +275,5 @@
 </joint>
 <joint name="lidar_left_joint" type="fixed">
-  <origin xyz="1.29 0.313 0.086" rpy="0 0 1.5707963"/>
+  <origin xyz="1.29 0.313 0.086" rpy="0 0 -1.5707963"/>
   <parent link="base_link"/>
   <child link="lidar_left_1"/>
